File: mk2/mk2/mk2.kicad_sch (KiCad schematic)
At the start: 19 parts, among them Q1 IRF540N, SW1 SW_Push, SW2 Switch_Slide_Top_CnK

Commit message: KiCad
Parts:
- added C11, C12: 35v 5600uF, symbol Device:C
- added D2: 1N5408 Flyback, symbol Device:D
- added L1: 161 Turn 18 AWG Coil, symbol Device:L
- C1, C10, C2, C3, C4, C5, C6, C7, C8, C9: value 25v 4900uF -> 35v 5600uF
- Q1: value IRF540N -> IRLZ44N
Connections:
- net COM: now reaches A2.4 (GND), BT2.2 (-), D1.1 (K), R1.2, R2.2
- net COM: now also C1.2, C10.2, C2.2, C3.2, C4.2, C5.2, C6.2, C7.2, C8.2, C9.2, Q1.3 (S), C11.2, C12.2
- removed net PWR_24V: C1.2, C10.2, C2.2, C3.2, C4.2, C5.2, C6.2, C7.2, C8.2, C9.2, Q1.2 (D)
- net PWR_GND renamed Load +
- net Load +: now also C11.1, C12.1, D2.1 (K), L1.1; no longer Q1.3 (S)
- new net Load -: D2.2 (A), L1.2, Q1.2 (D)
Other:
- note added: "0.85 in Projectile Length 2.55 in Coil Length"
- note added: "10x 35v 5600uF Electrolytic Capacitors 1x Arduino Nano 1x Electro Cookie Mini Protoboard 2x 10k Resistors 1x 330 Resistor 1x IRLZ44N Mosfet 1x Push Button 1x 9v Battery 1x Slide Switch 1x 1N5408 Diode 1x 161 Turn 18 AWG Coil"
- note added: "Coil"
- note added: "Notes"
- note removed: "10x 25v 4900uF Electrolytic Capacitors 1x Arduino Nano 1x Electro Cookie Mini Protoboard 2x 10k Resistors 1x 330 Resistor 1x IRF510N Mosfet 1x Push Button 1x 9v Battery 1x Slide Switch"
- company: Nicholas Niles & Jack Donnelly -> Nicholas Niles
- moved on the sheet: A2, BT2, C1, C10, C2, C3, C4, C5, C6, C7, C8, C9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
