File: mk2/main board/main board.kicad_pcb (KiCad board)
At the start: 2 copper layers, 40.6 x 59.7 mm, 6 parts, among them J1 Conn_01x02_Male, Q1 IRLZ44N

Commit message: PCB Updates
Parts:
- added J2: Conn_01x02_Male, Connector_PinHeader_2.54mm:PinHeader_1x02_P2.54mm_Horizontal, F.Cu at (125.0, 116.8)
- added SW1: SW_Push, Button_Switch_THT:SW_PUSH-12mm, F.Cu at (123.2, 97.3)
- moved J1 4.57 mm to (125.0, 123.8), turned to 180 degrees
Connections:
- A1 pad 13: unconnected-(A1-Pad13) -> Net-(A1-Pad13)
Routing:
- net Net-(A1-Pad13): track 0.00 -> 85.9 mm
- net Net-(A1-Pad29): track 88.3 -> 136.1 mm
- net Net-(A1-Pad30): track 11.6 -> 7.04 mm
Other:
- board size 40.6 x 59.7 mm -> 47 x 59.7 mm
