File: mk2/main board/main board.kicad_pcb (KiCad board)
At the start: 2 copper layers, 47 x 59.7 mm, 8 parts, among them J1 Conn_01x02_Male, J2 Conn_01x02_Male, Q1 IRLZ44N, SW1 SW_Push

Commit message: Work updates
Parts:
- added REF**: MountingHole_3.2mm_M3, MountingHole:MountingHole_3.2mm_M3, F.Cu at (156.8, 141.0)
- added REF**: MountingHole_3.2mm_M3, MountingHole:MountingHole_3.2mm_M3, F.Cu at (156.8, 88.9)
- added REF**: MountingHole_3.2mm_M3, MountingHole:MountingHole_3.2mm_M3, F.Cu at (117.5, 141.0)
- added REF**: MountingHole_3.2mm_M3, MountingHole:MountingHole_3.2mm_M3, F.Cu at (117.5, 88.9)
- moved R2 2.53 mm to (148.0, 124.5), turned to 0 degrees
Routing:
- net Net-(A1-Pad6): track 25.2 -> 19.8 mm
- net Net-(A1-Pad29): track 136.1 -> 140.3 mm
- net unconnected-(Q1-Pad2): track 27.3 -> 29.4 mm
Other:
- outline, holes or cut-outs redrawn

Commit message: Board Updates (Simplification)
Parts:
- removed REF** (x4): MountingHole_3.2mm_M3, MountingHole:MountingHole_3.2mm_M3
- removed SW1: SW_Push, Button_Switch_THT:SW_PUSH-12mm
- D1: footprint LED_THT:LED_D3.0mm -> fab:LED_1206
- R1: footprint Resistor_THT:R_Axial_DIN0207_L6.3mm_D2.5mm_P7.62mm_Horizontal -> fab:R_1206
- moved J1 10.2 mm to (124.5, 134.0), turned to -90 degrees
- moved R1 5.46 mm to (148.6, 99.7)
- moved J2 5.33 mm to (123.2, 121.8), turned to 90 degrees
- moved D1 2.40 mm to (148.6, 105.4)
Routing:
- net Net-(J1-Pin_2): track 140.3 -> 102.1 mm
- net Net-(A1-D10): track 85.9 -> 73.7 mm
- net Net-(A1-D4): track 6.19 -> 8.25 mm
- net Net-(A1-VIN): track 7.04 -> 8.93 mm
- net Net-(D1-K): track 2.85 -> 2.31 mm
Other:
- board size 47 x 59.7 mm -> 38.7 x 59.7 mm
- board text removed: "2"
- board text removed: "Ni"
