File: mk2/capacitor bank/capacitor bank.kicad_pcb (KiCad board)
At the start: 2 copper layers, 228.6 x 61 mm, 13 parts

Commit message: Work updates
Parts:
- moved C2 91.2 mm to (142.8, 58.4)
- moved C5 91.2 mm to (156.2, 81.5)
- moved C3 91.2 mm to (116.2, 58.4)
- moved C11 91.2 mm to (129.6, 81.5)
- moved C12 91.2 mm to (89.7, 58.4)
- moved C13 91.2 mm to (76.3, 81.5)
- moved C8 91.2 mm to (103.1, 81.5)
- moved C1 31.7 mm to (142.8, 105.5)
- moved C10 31.7 mm to (156.3, 128.6)
- moved C4 31.7 mm to (129.7, 128.6)
- moved C6 31.7 mm to (169.4, 105.5)
- moved C9 31.7 mm to (116.3, 105.5)
- moved C7 31.7 mm to (103.2, 128.6)
Routing:
- net Net-(C1-Pad2): track 345.7 -> 380.6 mm
- net Net-(C1-Pad1): track 355.0 -> 380.4 mm
Other:
- board size 228.6 x 61 mm -> 125.7 x 99.7 mm

Commit message: Board Updates (Simplification)
Other:
- board size 125.7 x 99.7 mm -> 121.3 x 99.9 mm
- board text removed: "2"
- board text removed: "Ni"
Changed lines of the file:
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@@
 			(drillshape 0)
 			(scaleselection 1)
-			(outputdirectory "../../../../Downloads/")
+			(outputdirectory "../../../../../../../../Downloads/")
 		)
 	)
@@
 	)
 	(gr_line
-		(start 179.07 137.955)
+		(start 174.625 137.795)
 		(end 63.5 137.955)
 		(stroke
@@
 	(gr_line
 		(start 63.5 38.26)
-		(end 179.07 38.26)
+		(end 174.625 38.1)
 		(stroke
 			(width 0.1)
@@
 	)
 	(gr_arc
-		(start 184.15 132.875)
-		(mid 182.662102 136.467102)
-		(end 179.07 137.955)
+		(start 179.705 132.715)
+		(mid 178.217102 136.307102)
+		(end 174.625 137.795)
 		(stroke
 			(width 0.1)
@@
 	)
 	(gr_arc
-		(start 179.07 38.26)
-		(mid 182.662102 39.747898)
-		(end 184.15 43.34)
+		(start 174.625 38.1)
+		(mid 178.217102 39.587898)
+		(end 179.705 43.18)
 		(stroke
 			(width 0.1)
@@
 	)
 	(gr_line
-		(start 184.15 43.34)
-		(end 184.15 132.875)
+		(start 179.705 43.18)
+		(end 179.705 132.715)
 		(stroke
 			(width 0.1)
@@
 		(layer "Edge.Cuts")
 	)
-	(gr_text "2"
-		(at 178.435 45.085 0)
-		(layer "F.Cu")
-		(effects
-			(font
-				(size 2.75 2.75)
-				(thickness 0.6875)
-			)
-		)
-	)
-	(gr_text "Ni"
-		(at 169.545 52.705 0)
-		(layer "F.Cu")
-		(effects
-			(font
-				(size 10 10)
-				(thickness 2)
-			)
-		)
-	)
 	(segment
 		(start 175.895 88.265)
 		(end 175.895 98.968)
-		(width 3)
+		(width 5)
 		(layer "F.Cu")
 		(net 1)
@@
 		(start 169.398 121.432)
 		(end 169.398 105.465)
-		(width 3)
+		(width 5)
 		(layer "F.Cu")
 		(net 1)
@@
 		(start 156.158629 81.509)
 		(end 156.195 81.545371)
-		(width 3)
+		(width 5)
 		(layer "F.Cu")
 		(net 1)
@@
 		(start 97.379742 128.576742)
 		(end 91.518 122.715)
-		(width 3)
+		(width 5)
 		(layer "F.Cu")
 		(net 1)
@@
 		(start 116.334371 105.501371)
 		(end 116.298 105.465)
-		(width 3)
+		(width 5)
 		(layer "F.Cu")
 		(net 1)
@@
 		(start 116.298 105.465)
 		(end 169.398 105.465)
-		(width 3)
+		(width 5)
 		(layer "F.Cu")
 		(net 1)
@@
 		(start 165.1 76.835)
 		(end 165.1 69.85)
-		(width 3)
+		(width 5)
 		(layer "F.Cu")
 		(net 1)
@@
 		(start 147.32 63.5)
 		(end 142.755 58.935)
-		(width 3)
+		(width 5)
 		(layer "F.Cu")
 		(net 1)
@@
 		(start 156.195 81.545371)
 		(end 160.389629 81.545371)
-		(width 3)
+		(width 5)
 		(layer "F.Cu")
 		(net 1)
@@
 		(start 169.175371 81.545371)
 		(end 175.895 88.265)
-		(width 3)
+		(width 5)
 		(layer "F.Cu")
 		(net 1)
@@
 		(start 76.263 81.509)
 		(end 156.158629 81.509)
-		(width 3)
+		(width 5)
 		(layer "F.Cu")
 		(net 1)
@@
 		(start 91.518 122.715)
 		(end 83.82 122.715)
-		(width 3)
+		(width 5)
 		(layer "F.Cu")
 		(net 1)
@@
 		(start 162.239629 128.590371)
 		(end 169.398 121.432)
-		(width 3)
+		(width 5)
 		(layer "F.Cu")
 		(net 1)
@@
 		(start 103.18 128.576742)
 		(end 97.379742 128.576742)
-		(width 3)
+		(width 5)
 		(layer "F.Cu")
 		(net 1)
@@
 		(start 103.18 128.576742)
 		(end 107.008258 128.576742)
-		(width 3)
+		(width 5)
 		(layer "F.Cu")
 		(net 1)
@@
 		(start 156.274371 128.576742)
 		(end 156.288 128.590371)
-		(width 3)
+		(width 5)
 		(layer "F.Cu")
 		(net 1)
@@
 		(start 158.75 63.5)
 		(end 147.32 63.5)
-		(width 3)
+		(width 5)
 		(layer "F.Cu")
 		(net 1)
@@
 		(start 160.389629 81.545371)
 		(end 169.175371 81.545371)
-		(width 3)
+		(width 5)
 		(layer "F.Cu")
 		(net 1)
@@
 		(start 160.389629 81.545371)
 		(end 165.1 76.835)
-		(width 3)
+		(width 5)
 		(layer "F.Cu")
 		(net 1)
@@
 		(start 175.895 98.968)
 		(end 169.398 105.465)
-		(width 3)
+		(width 5)
 		(layer "F.Cu")
 		(net 1)
@@
 		(start 156.288 128.590371)
 		(end 162.239629 128.590371)
-		(width 3)
+		(width 5)
 		(layer "F.Cu")
 		(net 1)
@@
 		(start 103.18 128.576742)
 		(end 156.274371 128.576742)
-		(width 3)
+		(width 5)
 		(layer "F.Cu")
 		(net 1)
@@
 		(start 89.655 58.42)
 		(end 142.755 58.42)
-		(width 3)
+		(width 5)
 		(layer "F.Cu")
 		(net 1)
@@
 		(start 142.755 58.935)
 		(end 142.755 58.42)
-		(width 3)
+		(width 5)
 		(layer "F.Cu")
 		(net 1)
@@
 		(start 165.1 69.85)
 		(end 158.75 63.5)
-		(width 3)
+		(width 5)
 		(layer "F.Cu")
 		(net 1)
@@
 		(start 103.18 105.973)
 		(end 106.758 102.395)
-		(width 3)
+		(width 5)
 		(layer "F.Cu")
 		(net 2)
@@
 		(start 93.98 102.395)
 		(end 93.98 97.155)
-		(width 3)
+		(width 5)
 		(layer "F.Cu")
 		(net 2)
@@
 		(start 71.12 88.9)
 		(end 66.675 84.455)
-		(width 3)
+		(width 5)
 		(layer "F.Cu")
 		(net 2)
@@
 		(start 116.298 95.465)
 		(end 169.398 95.465)
-		(width 3)
+		(width 5)
 		(layer "F.Cu")
 		(net 2)
@@
 		(start 93.98 102.395)
 		(end 83.82 102.395)
-		(width 3)
+		(width 5)
 		(layer "F.Cu")
 		(net 2)
@@
 		(start 89.655 48.42)
 		(end 142.755 48.42)
-		(width 3)
+		(width 5)
 		(layer "F.Cu")
 		(net 2)
@@
 		(start 85.725 88.9)
 		(end 71.12 88.9)
-		(width 3)
+		(width 5)
 		(layer "F.Cu")
 		(net 2)
@@
 		(start 109.259 99.894)
 		(end 109.22 99.855)
-		(width 3)
+		(width 5)
 		(layer "F.Cu")
 		(net 2)
@@
 		(start 156.195 71.545371)
 		(end 76.299371 71.545371)
-		(width 3)
+		(width 5)
 		(layer "F.Cu")
 		(net 2)
@@
 		(start 76.263 71.509)
 		(end 76.263 57.722)
-		(width 3)
+		(width 5)
 		(layer "F.Cu")
 		(net 2)
@@
 		(start 103.18 118.576742)
 		(end 156.274371 118.576742)
-		(width 3)
+		(width 5)
 		(layer "F.Cu")
 		(net 2)
@@
 		(start 85.565 48.42)
 		(end 89.655 48.42)
-		(width 3)
+		(width 5)
 		(layer "F.Cu")
 		(net 2)
@@
 		(start 76.299371 71.545371)
 		(end 76.263 71.509)
-		(width 3)
+		(width 5)
 		(layer "F.Cu")
 		(net 2)
@@
 		(start 66.675 84.455)
 		(end 66.675 76.835)
-		(width 3)
+		(width 5)
 		(layer "F.Cu")
 		(net 2)
@@
 		(start 106.758 102.395)
 		(end 107.989 101.164)
-		(width 3)
+		(width 5)
 		(layer "F.Cu")
 		(net 2)
@@
 		(start 113.688 95.465)
 		(end 116.298 95.465)
-		(width 3)
+		(width 5)
 		(layer "F.Cu")
 		(net 2)
@@
 		(start 103.18 118.576742)
 		(end 103.18 105.973)
-		(width 3)
+		(width 5)
 		(layer "F.Cu")
 		(net 2)
@@
 		(start 107.989 101.164)
 		(end 109.259 99.894)
-		(width 3)
+		(width 5)
 		(layer "F.Cu")
 		(net 2)
@@
 		(start 76.263 57.722)
 		(end 85.565 48.42)
-		(width 3)
+		(width 5)
 		(layer "F.Cu")
 		(net 2)
@@
 		(start 72.001 71.509)
 		(end 76.263 71.509)
-		(width 3)
+		(width 5)
 		(layer "F.Cu")
 		(net 2)
@@
 		(start 93.98 97.155)
 		(end 85.725 88.9)
-		(width 3)
+		(width 5)
 		(layer "F.Cu")
 		(net 2)
@@
 		(start 109.259 99.894)
 		(end 113.688 95.465)
-		(width 3)
+		(width 5)
 		(layer "F.Cu")
 		(net 2)
@@
 		(start 156.274371 118.576742)
 		(end 156.288 118.590371)
-		(width 3)
+		(width 5)
 		(layer "F.Cu")
 		(net 2)
@@
 		(start 106.758 102.395)
 		(end 93.98 102.395)
-		(width 3)
+		(width 5)
 		(layer "F.Cu")
 		(net 2)
@@
 		(start 66.675 76.835)
 		(end 72.001 71.509)
-		(width 3)
+		(width 5)
 		(layer "F.Cu")
 		(net 2)
